File: KiCad/croissant.kicad_sch (KiCad schematic)
At the start: 52 parts, among them J1 USB_C_Receptacle_PowerOnly_6P, Q1 NMOS, SW1 SW_SPST, U1 NE556, U2 TL064, U3 TL064

Commit message: Specify component values
Parts:
- C2: value C -> 22n
- C3, C4, C7: value C -> 0.1u
- C5: value C -> 5n
- C6: value C -> 1u
- R1: value R -> 18k
- R10, R11, R12, R13, R14, R15, R16, R17, R18, R19, R20, R21, R22, R23, R9: value R -> 1k
- R2: value R -> 82k
- R3, R4: value R -> 10k
- R5: value R -> 100k
- R6: value R -> 6k8
- R7: value R -> 4k7
- R8: value R -> 680k
Changed lines of the file:
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@@
       (effects (font (size 1.27 1.27)))
     )
-    (property "Value" "C" (at 266.7 104.14 90)
+    (property "Value" "0.1u" (at 266.7 104.14 90)
       (effects (font (size 1.27 1.27)))
     )
@@
       (effects (font (size 1.27 1.27)))
     )
-    (property "Value" "R" (at 147.32 140.97 90)
+    (property "Value" "4k7" (at 147.32 140.97 90)
       (effects (font (size 1.27 1.27)))
     )
@@
       (effects (font (size 1.27 1.27)) (justify left))
     )
-    (property "Value" "R" (at 182.88 50.165 0)
+    (property "Value" "1k" (at 182.88 50.165 0)
       (effects (font (size 1.27 1.27)) (justify left))
     )
@@
       (effects (font (size 1.27 1.27)) (justify left))
     )
-    (property "Value" "R" (at 111.76 60.325 0)
+    (property "Value" "10k" (at 111.76 60.325 0)
       (effects (font (size 1.27 1.27)) (justify left))
     )
@@
       (effects (font (size 1.27 1.27)) (justify left))
     )
-    (property "Value" "R" (at 236.22 50.165 0)
+    (property "Value" "1k" (at 236.22 50.165 0)
       (effects (font (size 1.27 1.27)) (justify left))
     )
@@
       (effects (font (size 1.27 1.27)) (justify left))
     )
-    (property "Value" "R" (at 245.11 50.165 0)
+    (property "Value" "1k" (at 245.11 50.165 0)
       (effects (font (size 1.27 1.27)) (justify left))
     )
@@
       (effects (font (size 1.27 1.27)))
     )
-    (property "Value" "C" (at 163.83 113.03 90)
+    (property "Value" "1u" (at 163.83 113.03 90)
       (effects (font (size 1.27 1.27)))
     )
@@
       (effects (font (size 1.27 1.27)) (justify left))
     )
-    (property "Value" "R" (at 182.88 74.295 0)
+    (property "Value" "1k" (at 182.88 74.295 0)
       (effects (font (size 1.27 1.27)) (justify left))
     )
@@
       (effects (font (size 1.27 1.27)) (justify left))
     )
-    (property "Value" "R" (at 111.76 70.485 0)
+    (property "Value" "10k" (at 111.76 70.485 0)
       (effects (font (size 1.27 1.27)) (justify left))
     )
@@
       (effects (font (size 1.27 1.27)) (justify right))
     )
-    (property "Value" "C" (at 243.84 142.875 0)
+    (property "Value" "5n" (at 243.84 142.875 0)
       (effects (font (size 1.27 1.27)) (justify right))
     )
@@
       (effects (font (size 1.27 1.27)) (justify left))
     )
-    (property "Value" "R" (at 209.55 74.295 0)
+    (property "Value" "1k" (at 209.55 74.295 0)
       (effects (font (size 1.27 1.27)) (justify left))
     )
@@
       (effects (font (size 1.27 1.27)) (justify left))
     )
-    (property "Value" "R" (at 227.33 74.295 0)
+    (property "Value" "1k" (at 227.33 74.295 0)
       (effects (font (size 1.27 1.27)) (justify left))
     )
@@
       (effects (font (size 1.27 1.27)))
     )
-    (property "Value" "R" (at 243.84 129.54 90)
+    (property "Value" "100k" (at 243.84 129.54 90)
       (effects (font (size 1.27 1.27)))
     )
@@
       (effects (font (size 1.27 1.27)) (justify right))
     )
-    (property "Value" "C" (at 67.31 145.415 0)
+    (property "Value" "22n" (at 67.31 145.415 0)
       (effects (font (size 1.27 1.27)) (justify right))
     )
@@
       (effects (font (size 1.27 1.27)))
     )
-    (property "Value" "R" (at 143.51 121.92 90)
+    (property "Value" "680k" (at 143.51 121.92 90)
       (effects (font (size 1.27 1.27)))
     )
@@
       (effects (font (size 1.27 1.27)) (justify left))
     )
-    (property "Value" "R" (at 191.77 50.165 0)
+    (property "Value" "1k" (at 191.77 50.165 0)
       (effects (font (size 1.27 1.27)) (justify left))
     )
@@
       (effects (font (size 1.27 1.27)) (justify left))
     )
-    (property "Value" "R" (at 66.04 137.795 0)
+    (property "Value" "18k" (at 66.04 137.795 0)
       (effects (font (size 1.27 1.27)) (justify left))
     )
@@
       (effects (font (size 1.27 1.27)) (justify left))
     )
-    (property "Value" "R" (at 138.43 137.795 0)
+    (property "Value" "6k8" (at 138.43 137.795 0)
       (effects (font (size 1.27 1.27)) (justify left))
     )
@@
       (effects (font (size 1.27 1.27)) (justify left))
     )
-    (property "Value" "R" (at 209.55 50.165 0)
+    (property "Value" "1k" (at 209.55 50.165 0)
       (effects (font (size 1.27 1.27)) (justify left))
     )
@@
       (effects (font (size 1.27 1.27)) (justify left))
     )
-    (property "Value" "R" (at 227.33 50.165 0)
+    (property "Value" "1k" (at 227.33 50.165 0)
       (effects (font (size 1.27 1.27)) (justify left))
     )
@@
       (effects (font (size 1.27 1.27)))
     )
-    (property "Value" "C" (at 90.17 54.61 90)
+    (property "Value" "0.1u" (at 90.17 54.61 90)
       (effects (font (size 1.27 1.27)))
     )
@@
       (effects (font (size 1.27 1.27)))
     )
-    (property "Value" "R" (at 69.85 129.54 90)
+    (property "Value" "82k" (at 69.85 129.54 90)
       (effects (font (size 1.27 1.27)))
     )
@@
       (effects (font (size 1.27 1.27)))
     )
-    (property "Value" "C" (at 227.33 113.03 90)
+    (property "Value" "0.1u" (at 227.33 113.03 90)
       (effects (font (size 1.27 1.27)))
     )
@@
       (effects (font (size 1.27 1.27)) (justify left))
     )
-    (property "Value" "R" (at 218.44 50.165 0)
+    (property "Value" "1k" (at 218.44 50.165 0)
       (effects (font (size 1.27 1.27)) (justify left))
     )
@@
       (effects (font (size 1.27 1.27)) (justify left))
     )
-    (property "Value" "R" (at 218.44 74.295 0)
+    (property "Value" "1k" (at 218.44 74.295 0)
       (effects (font (size 1.27 1.27)) (justify left))
     )
@@
       (effects (font (size 1.27 1.27)) (justify left))
     )
-    (property "Value" "R" (at 200.66 74.295 0)
+    (property "Value" "1k" (at 200.66 74.295 0)
       (effects (font (size 1.27 1.27)) (justify left))
     )
@@
       (effects (font (size 1.27 1.27)) (justify left))
     )
-    (property "Value" "R" (at 236.22 74.295 0)
+    (property "Value" "1k" (at 236.22 74.295 0)
       (effects (font (size 1.27 1.27)) (justify left))
     )
@@
       (effects (font (size 1.27 1.27)) (justify left))
     )
-    (property "Value" "R" (at 191.77 74.295 0)
+    (property "Value" "1k" (at 191.77 74.295 0)
       (effects (font (size 1.27 1.27)) (justify left))
     )
@@
       (effects (font (size 1.27 1.27)) (justify left))
     )
-    (property "Value" "R" (at 200.66 50.165 0)
-      (effects (font (size 1.27 1.27)) (justify left))
-    )
+    (property "Value" "1k" (at 200.66 50.165 0)
+      (effects (font (size 1.27 1.27)) (justify left))
+    )

Commit message: Fix designator
Parts:
- U1: footprint (none) -> Package_SO:SOIC-14_3.9x8.7mm_P1.27mm
- renumbered U3 to U2
Changed lines of the file:
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@@
   (symbol (lib_id "Amplifier_Operational:TL064") (at 88.9 67.31 0) (unit 5)
     (in_bom yes) (on_board yes) (dnp no) (fields_autoplaced)
-    (property "Reference" "U3" (at 87.63 66.675 0)
+    (property "Reference" "U2" (at 87.63 66.675 0)
       (effects (font (size 1.27 1.27)) (justify left))
     )
@@
       (project "croissant"
         (path "/9d4c4425-9345-4751-a711-72e95f2cc96d"
-          (reference "U3") (unit 5)
+          (reference "U2") (unit 5)
         )
       )
@@
       (effects (font (size 1.27 1.27)) (justify left))
     )
-    (property "Footprint" "" (at 223.52 132.08 0)
+    (property "Footprint" "Package_SO:SOIC-14_3.9x8.7mm_P1.27mm" (at 223.52 132.08 0)
       (effects (font (size 1.27 1.27)) hide)
     )
@@
       (effects (font (size 1.27 1.27)) (justify left))
     )
-    (property "Footprint" "" (at 45.72 132.08 0)
-      (effects (font (size 1.27 1.27)) hide)
-    )
+    (property "Footprint" "Package_SO:SOIC-14_3.9x8.7mm_P1.27mm" (at 45.72 132.08 0)
+      (effects (font (size 1.27 1.27)) hide)
+    )
