File: KiCad/croissant.kicad_sch (KiCad schematic)
At the start: 53 parts, among them J1 USB_C_Receptacle_PowerOnly_6P, Q1 NMOS, SW1 SW_SPDT, U1 NE556, U2 TL064

Commit message: Advance routing
Parts:
- C1: value C -> 0.1u
Connections:
- net +5V: no longer C4.1
- net GND: now also C4.1; no longer C4.2
- net at U1.3 (CV): now also C4.2
- no-connect marks 7 -> 6
Changed lines of the file:
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@@
   (junction (at 261.62 121.92) (diameter 0) (color 0 0 0 0)
   )
-  (junction (at 222.25 121.92) (diameter 0) (color 0 0 0 0)
-  )
   (junction (at 198.12 44.45) (diameter 0) (color 0 0 0 0)
   )
@@
   )
   (no_connect (at 133.35 43.18))
-  (no_connect (at 33.02 132.08))
   (no_connect (at 118.11 40.64))
   (no_connect (at 118.11 45.72))
@@
     (stroke (width 0) (type default))
   )
-  (wire (pts (xy 222.25 121.92) (xy 222.25 127))
-    (stroke (width 0) (type default))
-  )
   (wire (pts (xy 59.69 137.16) (xy 58.42 137.16))
     (stroke (width 0) (type default))
@@
   )
   (wire (pts (xy 180.34 44.45) (xy 189.23 44.45))
-    (stroke (width 0) (type default))
-  )
-  (wire (pts (xy 222.25 119.38) (xy 222.25 121.92))
     (stroke (width 0) (type default))
   )
@@
     )
   )
+  (symbol (lib_id "Device:C") (at 29.21 132.08 90) (unit 1)
+    (in_bom yes) (on_board yes) (dnp no) (fields_autoplaced)
+    (property "Reference" "C4" (at 29.21 125.73 90)
+      (effects (font (size 1.27 1.27)))
+    )
+    (property "Value" "0.1u" (at 29.21 128.27 90)
+      (effects (font (size 1.27 1.27)))
+    )
+    (property "Footprint" "Capacitor_SMD:C_0603_1608Metric" (at 33.02 131.1148 0)
+      (effects (font (size 1.27 1.27)) hide)
+    )
+    (property "Datasheet" "~" (at 29.21 132.08 0)
+      (effects (font (size 1.27 1.27)) hide)
+    )
+    (pin "1")
+    (pin "2")
+    (instances
+      (project "croissant"
+        (path "/9d4c4425-9345-4751-a711-72e95f2cc96d"
+          (reference "C4") (unit 1)
+        )
+      )
+    )
+  )
   (symbol (lib_id "Device:R") (at 180.34 48.26 0) (unit 1)
     (in_bom yes) (on_board yes) (dnp no) (fields_autoplaced)
@@
         (path "/9d4c4425-9345-4751-a711-72e95f2cc96d"
           (reference "R9") (unit 1)
-        )
-      )
-    )
-  )
-  (symbol (lib_id "power:GND") (at 229.87 121.92 90) (unit 1)
-    (in_bom yes) (on_board yes) (dnp no) (fields_autoplaced)
-    (property "Reference" "#PWR017" (at 236.22 121.92 0)
-      (effects (font (size 1.27 1.27)) hide)
-    )
-    (property "Value" "GND" (at 233.68 122.555 90)
-      (effects (font (size 1.27 1.27)) (justify right))
-    )
-    (property "Footprint" "" (at 229.87 121.92 0)
-      (effects (font (size 1.27 1.27)) hide)
-    )
-    (property "Datasheet" "" (at 229.87 121.92 0)
-      (effects (font (size 1.27 1.27)) hide)
-    )
-    (pin "1")
-    (instances
-      (project "croissant"
-        (path "/9d4c4425-9345-4751-a711-72e95f2cc96d"
-          (reference "#PWR017") (unit 1)
         )
       )
@@
     )
   )
+  (symbol (lib_id "power:GND") (at 25.4 132.08 270) (unit 1)
+    (in_bom yes) (on_board yes) (dnp no) (fields_autoplaced)
+    (property "Reference" "#PWR017" (at 19.05 132.08 0)
+      (effects (font (size 1.27 1.27)) hide)
+    )
+    (property "Value" "GND" (at 21.59 131.445 90)
+      (effects (font (size 1.27 1.27)) (justify right))
+    )
+    (property "Footprint" "" (at 25.4 132.08 0)
+      (effects (font (size 1.27 1.27)) hide)
+    )
+    (property "Datasheet" "" (at 25.4 132.08 0)
+      (effects (font (size 1.27 1.27)) hide)
+    )
+    (pin "1")
+    (instances
+      (project "croissant"
+        (path "/9d4c4425-9345-4751-a711-72e95f2cc96d"
+          (reference "#PWR017") (unit 1)
+        )
+      )
+    )
+  )
   (symbol (lib_id "power:GND") (at 207.01 83.82 0) (unit 1)
     (in_bom yes) (on_board yes) (dnp no) (fields_autoplaced)
@@
     )
   )
-  (symbol (lib_id "power:+5V") (at 222.25 119.38 0) (unit 1)
-    (in_bom yes) (on_board yes) (dnp no) (fields_autoplaced)
-    (property "Reference" "#PWR05" (at 222.25 123.19 0)
-      (effects (font (size 1.27 1.27)) hide)
-    )
-    (property "Value" "+5V" (at 222.25 115.57 0)
-      (effects (font (size 1.27 1.27)))
-    )
-    (property "Footprint" "" (at 222.25 119.38 0)
-      (effects (font (size 1.27 1.27)) hide)
-    )
-    (property "Datasheet" "" (at 222.25 119.38 0)
+  (symbol (lib_id "power:+5V") (at 222.25 127 0) (unit 1)
+    (in_bom yes) (on_board yes) (dnp no) (fields_autoplaced)
+    (property "Reference" "#PWR05" (at 222.25 130.81 0)
+      (effects (font (size 1.27 1.27)) hide)
+    )
+    (property "Value" "+5V" (at 222.25 123.19 0)
+      (effects (font (size 1.27 1.27)))
+    )
+    (property "Footprint" "" (at 222.25 127 0)
+      (effects (font (size 1.27 1.27)) hide)
+    )
+    (property "Datasheet" "" (at 222.25 127 0)
       (effects (font (size 1.27 1.27)) hide)
     )
@@
         (path "/9d4c4425-9345-4751-a711-72e95f2cc96d"
           (reference "#PWR07") (unit 1)
-        )
-      )
-    )
-  )
-  (symbol (lib_id "Device:C") (at 226.06 121.92 90) (unit 1)
-    (in_bom yes) (on_board yes) (dnp no) (fields_autoplaced)
-    (property "Reference" "C4" (at 226.06 115.57 90)
-      (effects (font (size 1.27 1.27)))
-    )
-    (property "Value" "0.1u" (at 226.06 118.11 90)
-      (effects (font (size 1.27 1.27)))
-    )
-    (property "Footprint" "Capacitor_SMD:C_0603_1608Metric" (at 229.87 120.9548 0)
-      (effects (font (size 1.27 1.27)) hide)
-    )
-    (property "Datasheet" "~" (at 226.06 121.92 0)
-      (effects (font (size 1.27 1.27)) hide)
-    )
-    (pin "1")
-    (pin "2")
-    (instances
-      (project "croissant"
-        (path "/9d4c4425-9345-4751-a711-72e95f2cc96d"
-          (reference "C4") (unit 1)
         )
       )
@@
       (effects (font (size 1.27 1.27)))
     )
-    (property "Value" "C" (at 52.07 109.22 90)
-      (effects (font (size 1.27 1.27)))
-    )
+    (property "Value" "0.1u" (at 52.07 109.22 90)
+      (effects (font (size 1.27 1.27)))
+    )
