File: KiCad/croissant.kicad_pcb (KiCad board)
At the start: 2 copper layers, 149.8 x 90.3 mm, 54 parts, among them J1 USB_C_Receptacle_PowerOnly_6P, Q1 NMOS, SW1 SW_SPDT, U1 NE556, U2 TL064

Commit message: Add JLC reference placeholder
Other:
- board text added: "JLCJLCJLCJLC"
Changed lines of the file:
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@@
       (plot_on_all_layers_selection 0x0000000_00000000)
       (disableapertmacros false)
-      (usegerberextensions false)
+      (usegerberextensions true)
       (usegerberattributes true)
-      (usegerberadvancedattributes true)
-      (creategerberjobfile true)
+      (usegerberadvancedattributes false)
+      (creategerberjobfile false)
       (dashed_line_dash_ratio 12.000000)
       (dashed_line_gap_ratio 3.000000)
@@
       (psa4output false)
       (plotreference true)
-      (plotvalue true)
+      (plotvalue false)
       (plotinvisibletext false)
       (sketchpadsonfab false)
-      (subtractmaskfromsilk false)
+      (subtractmaskfromsilk true)
       (outputformat 1)
       (mirror false)
-      (drillshape 1)
+      (drillshape 0)
       (scaleselection 1)
-      (outputdirectory "")
+      (outputdirectory "croissant-output/")
     )
   )
@@
     )
     (stroke (width 0.02928) (type solid)) (fill none) (layer "Edge.Cuts"))
+  (gr_text "JLCJLCJLCJLC" (at 150.5 98.5) (layer "B.SilkS")
+    (effects (font (size 1 1) (thickness 0.2) bold) (justify left bottom mirror))
+  )
   (segment (start 147.36 61) (end 147.32 60.96) (width 0.25) (layer "B.Cu") (net 1))
   (segment (start 151.35 73.66) (end 151.35 76.9) (width 0.25) (layer "B.Cu") (net 1))

Commit message: Add RefBoard on silkscreen
Other:
- board text added: "${RefBoard}"
Changed lines of the file:
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@@
     (effects (font (size 1 1) (thickness 0.2) bold) (justify left bottom mirror))
+  )
+  (gr_text "${RefBoard}" (at 149.25 102.25) (layer "B.SilkS")
+    (effects (font (size 1 1) (thickness 0.15)) (justify left bottom mirror))
   )
   (segment (start 147.36 61) (end 147.32 60.96) (width 0.25) (layer "B.Cu") (net 1))
